Commit message: Add new calubration config and urdf

File: z1_calibration/xacro/uncalibrated_robot.xacro (robot description, xacro)
@@ -226,9 +226,15 @@
     </link>
     <joint name="joint_ee" type="fixed">
-        <origin rpy="0 ${PI/2.0} 0" xyz="0.051 0.0 0.0"/>
+        <origin rpy="0 ${PI/2} 0" xyz="0.051 0.0 0.0"/>
             <parent link="link06"/>
         <child link="ee_link"/>
     </joint>
     <link name="ee_link"/>
+    <joint name="joint_checkerboard" type="fixed">
+        <origin rpy="${PI} 0 ${PI/2}" xyz="0 0.0 0.0"/>
+            <parent link="ee_link"/>
+        <child link="checkerboard_link"/>
+    </joint>
+    <link name="checkerboard_link"/>
     <xacro:if value="$(arg UnitreeGripper)">
         <joint name="gripperStator" type="fixed">

Commit message: a lot of params changed

File: z1_calibration/xacro/uncalibrated_robot.xacro (robot description, xacro)
@@ -12,5 +12,5 @@
     </joint>
     <joint name="static_camera_rgb_joint" type="fixed">
-        <origin rpy="0 0 0" xyz="0 1 2"/>
+        <origin rpy="0 0 0" xyz="0.85 -0.5 0.55"/>
         <parent link="world"/>
         <child link="camera_link"/>
